File: pcb/FloppyEmuButtonPanel.kicad_pcb (KiCad board)
At the start: 2 copper layers, 45.3 x 33.9 mm, 13 parts, among them J1 ButtonPanel, SW1 PREVIOUS/UP, SW2 SELECT, SW3 NEXT/DOWN, SW4 RESET

Commit message: PCB Update
Parts:
- J1: value ButtonPanel -> ButtonPanelConnector
- moved H1 0.06 mm to (102.3, 96.2)
- moved H2 0.06 mm to (102.3, 70.8)
- moved H3 0.06 mm to (140.4, 70.8)
- moved H4 0.06 mm to (140.4, 96.2)
Routing:
- net /NEXT: track 19.0 -> 20.9 mm
Other:
- board size 45.3 x 33.9 mm -> 45.3 x 33.3 mm
- board text added: "FloppyEmu Button Panel github.com/ThorstenBr/ FloppyEmuDiskIIEnclosure"
- board text added: "v1.0, 05/2022"
Changed lines of the file:
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@@
   (general
     (thickness 1.6)
-    (drawings 9)
-    (tracks 53)
+    (drawings 13)
+    (tracks 57)
     (zones 0)
     (modules 13)
@@
   )
   (module Mounting_Holes:MountingHole_3.2mm_M3 (layer F.Cu)
-    (at 140.462 96.266)
+    (at 140.41 96.23)
     (descr "Mounting Hole 3.2mm, no annular, M3")
     (tags "mounting hole 3.2mm no annular m3")
@@
   )
   (module Mounting_Holes:MountingHole_3.2mm_M3 (layer F.Cu)
-    (at 140.462 70.866)
+    (at 140.41 70.83)
     (descr "Mounting Hole 3.2mm, no annular, M3")
     (tags "mounting hole 3.2mm no annular m3")
@@
   )
   (module Mounting_Holes:MountingHole_3.2mm_M3 (layer F.Cu)
-    (at 102.362 70.866)
+    (at 102.31 70.83)
     (descr "Mounting Hole 3.2mm, no annular, M3")
     (tags "mounting hole 3.2mm no annular m3")
@@
   )
   (module Mounting_Holes:MountingHole_3.2mm_M3 (layer F.Cu)
-    (at 102.362 96.266)
+    (at 102.31 96.23)
     (descr "Mounting Hole 3.2mm, no annular, M3")
     (tags "mounting hole 3.2mm no annular m3")
@@
     (descr http://www.farnell.com/datasheets/1520732.pdf)
     (tags "connector multicomp MC9A MC9A12")
-    (fp_text reference J1 (at 13.843 -4.699) (layer B.SilkS)
-      (effects (font (size 1 1) (thickness 0.15)) (justify mirror))
-    )
-    (fp_text value ButtonPanel (at 4.699 -4.953) (layer F.Fab)
-      (effects (font (size 1 1) (thickness 0.15)))
+    (fp_text reference J1 (at -4.064 7.493) (layer B.SilkS)
+      (effects (font (size 1 1) (thickness 0.15)) (justify mirror))
+    )
+    (fp_text value ButtonPanelConnector (at 4.699 -4.953) (layer B.Paste) hide
+      (effects (font (size 1 1) (thickness 0.15)) (justify mirror))
     )
     (fp_line (start 15.75 -3.7) (end -5.55 -3.7) (layer B.CrtYd) (width 0.05))
@@
     )
   )
+  (gr_text "v1.0, 05/2022" (at 120.27 95.7) (layer F.SilkS)
+    (effects (font (size 1 1) (thickness 0.15)) (justify left))
+  )
+  (dimension 12.7 (width 0.15) (layer Dwgs.User)
+    (gr_text "12,700 mm" (at 134.06 64.25) (layer Dwgs.User)
+      (effects (font (size 1 1) (thickness 0.15)))
+    )
+    (feature1 (pts (xy 127.71 70.88) (xy 127.71 64.963579)))
+    (feature2 (pts (xy 140.41 70.88) (xy 140.41 64.963579)))
+    (crossbar (pts (xy 140.41 65.55) (xy 127.71 65.55)))
+    (arrow1a (pts (xy 127.71 65.55) (xy 128.836504 64.963579)))
+    (arrow1b (pts (xy 127.71 65.55) (xy 128.836504 66.136421)))
+    (arrow2a (pts (xy 140.41 65.55) (xy 139.283496 64.963579)))
+    (arrow2b (pts (xy 140.41 65.55) (xy 139.283496 66.136421)))
+  )
+  (dimension 12.7 (width 0.15) (layer Dwgs.User)
+    (gr_text "12,700 mm" (at 108.66 64.2) (layer Dwgs.User)
+      (effects (font (size 1 1) (thickness 0.15)))
+    )
+    (feature1 (pts (xy 102.31 70.83) (xy 102.31 64.913579)))
+    (feature2 (pts (xy 115.01 70.83) (xy 115.01 64.913579)))
+    (crossbar (pts (xy 115.01 65.5) (xy 102.31 65.5)))
+    (arrow1a (pts (xy 102.31 65.5) (xy 103.436504 64.913579)))
+    (arrow1b (pts (xy 102.31 65.5) (xy 103.436504 66.086421)))
+    (arrow2a (pts (xy 115.01 65.5) (xy 113.883496 64.913579)))
+    (arrow2b (pts (xy 115.01 65.5) (xy 113.883496 66.086421)))
+  )
+  (gr_text "FloppyEmu Button Panel\ngithub.com/ThorstenBr/\nFloppyEmuDiskIIEnclosure" (at 120.142 91.948) (layer F.SilkS)
+    (effects (font (size 1 1) (thickness 0.15)) (justify left))
+  )
   (dimension 12.7 (width 0.15) (layer Dwgs.User)
     (gr_text "12,700 mm" (at 93.696 89.88 270) (layer Dwgs.User)
@@
     (arrow2b (pts (xy 150.114 70.866) (xy 150.700421 71.992504)))
   )
-  (gr_line (start 144.018 67.183) (end 98.679 67.183) (layer Edge.Cuts) (width 0.05))
-  (gr_line (start 144.018 101.092) (end 144.018 67.183) (layer Edge.Cuts) (width 0.05))
-  (gr_line (start 98.679 101.092) (end 144.018 101.092) (layer Edge.Cuts) (width 0.05))
-  (gr_line (start 98.679 67.183) (end 98.679 101.092) (layer Edge.Cuts) (width 0.05))
+  (gr_line (start 144.018 66.9) (end 98.679 66.9) (layer Edge.Cuts) (width 0.05))
+  (gr_line (start 144.018 100.2) (end 144.018 66.9) (layer Edge.Cuts) (width 0.05))
+  (gr_line (start 98.679 100.2) (end 144.018 100.2) (layer Edge.Cuts) (width 0.05))
+  (gr_line (start 98.679 66.9) (end 98.679 100.2) (layer Edge.Cuts) (width 0.05))
   (segment (start 136.906 81.28) (end 136.906 82.423) (width 0.5) (layer F.Cu) (net 1))
   (segment (start 133.604 77.978) (end 136.906 81.28) (width 0.5) (layer F.Cu) (net 1))
@@
   (segment (start 129.286 84.963) (end 129.286 86.614) (width 0.5) (layer F.Cu) (net 6))
   (segment (start 129.286 86.614) (end 128.397 87.503) (width 0.5) (layer F.Cu) (net 6))
-  (segment (start 124.483 87.503) (end 118.26 81.28) (width 0.5) (layer F.Cu) (net 6))
-  (segment (start 128.397 87.503) (end 124.483 87.503) (width 0.5) (layer F.Cu) (net 6))
-  (segment (start 126.746 85.494) (end 118.26 93.98) (width 0.5) (layer B.Cu) (net 7))
+  (segment (start 125.857 87.462787) (end 125.857 87.503) (width 0.5) (layer F.Cu) (net 6))
+  (segment (start 119.674213 81.28) (end 125.857 87.462787) (width 0.5) (layer F.Cu) (net 6))
+  (segment (start 118.26 81.28) (end 119.674213 81.28) (width 0.5) (layer F.Cu) (net 6))
+  (segment (start 128.397 87.503) (end 125.857 87.503) (width 0.5) (layer F.Cu) (net 6))
   (segment (start 126.746 84.963) (end 126.746 85.494) (width 0.5) (layer B.Cu) (net 7))
   (segment (start 118.26 93.98) (end 111.76 93.98) (width 0.5) (layer B.Cu) (net 7))
+  (segment (start 118.26 93.98) (end 118.26 90.782) (width 0.5) (layer B.Cu) (net 7))
+  (segment (start 123.571 85.471) (end 126.746 85.471) (width 0.5) (layer B.Cu) (net 7))
+  (segment (start 118.26 90.782) (end 123.571 85.471) (width 0.5) (layer B.Cu) (net 7))
   (segment (start 104.775 79.121) (end 105.918 77.978) (width 0.5) (layer B.Cu) (net 8))
   (segment (start 102.489 79.121) (end 104.775 79.121) (width 0.5) (layer B.Cu) (net 8))
@@
     (polygon
       (pts
-        (xy 143.764 100.838) (xy 98.806 100.838) (xy 98.806 67.31) (xy 143.764 67.31)
+        (xy 144 100.2) (xy 98.7 100.2) (xy 98.7 66.9) (xy 144 66.9)
       )
     )
@@
     (polygon
       (pts
-        (xy 143.764 100.838) (xy 98.806 100.838) (xy 98.806 67.31) (xy 143.764 67.31)
+        (xy 144 100.2) (xy 98.7 100.2) (xy 98.7 66.9) (xy 144 66.9)
       )
     )
